File: main_board/main_board.kicad_sch (KiCad schematic)
At the start: 57 parts, among them J1 USB4105-GF-A-060, J2 Conn_01x06_Pin, Q3 NX3008PBK,215, U1 SSD1306, U2 ESP32-S2-SOLO, U3 TLV62568PDRLT, U4 MCP73832, U5 DW01, U6 8205A, U7 MAX17055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

Commit message: fix package issue on bom
Parts:
- U4: LCSC Part # C511264 -> C38066; MPN MCP73832T-2ACI/MC -> MCP73832T-2ACI/OT
Changed lines of the file:
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@@
       (effects (font (size 1.27 1.27)) hide)
     )
-    (property "LCSC Part #" "C511264" (at 33.02 123.19 0)
+    (property "LCSC Part #" "C38066" (at 33.02 123.19 0)
       (effects (font (size 1.27 1.27)) hide)
     )
-    (property "MPN" "MCP73832T-2ACI/MC" (at 33.02 123.19 0)
+    (property "MPN" "MCP73832T-2ACI/OT" (at 33.02 123.19 0)
       (effects (font (size 1.27 1.27)) hide)
     )
